File: sektoriloisto.sch (EAGLE design)
At the start: 0 parts

Commit message: Schematic added
Parts:
- added LED1, LED2, LED3, LED4, LED5, LED6: (no value), adafruit:LED5MM
- added R1, R2, R3, R4, R5, R6: (no value), rcl:R-EU_0207/10
- added T1, T2, T3, T4, T5, T6: 2N2222, adafruit:2N2222
- added U$1: ARDUINO-NOHOLE, adafruit:ARDUINO-NOHOLE
Connections:
- new net GND: T1.E, T2.E, T3.E, T4.E, T5.E, T6.E, U$1.GND1, U$1.GND2
- new net N$1: LED1.A, R1.1
- new net N$10: LED4.C, T4.C
- new net N$11: LED5.C, T5.C
- new net N$12: LED6.C, T6.C
- new net N$13: T1.B, U$1.D11
- new net N$14: T2.B, U$1.D10
- new net N$15: T3.B, U$1.D9
- new net N$16: T4.B, U$1.D6
- new net N$17: T5.B, U$1.D5
- new net N$18: T6.B, U$1.D4
- new net N$2: LED2.A, R2.1
- new net N$3: LED3.A, R3.1
- new net N$4: LED4.A, R4.1
- new net N$5: LED5.A, R5.1
- new net N$6: LED6.A, R6.1
- new net N$7: LED1.C, T1.C
- new net N$8: LED2.C, T2.C
- new net N$9: LED3.C, T3.C
- new net VCC: R1.2, R2.2, R3.2, R4.2, R5.2, R6.2, U$1.VIN
